File: RGBSystemTuner-PSU/RGBSystemTuner-PSU.kicad_sch (KiCad schematic)
At the start: 43 parts, among them IC701 78012AP, IC702 78012AP, IC703 78005AP, IC704 78009AP, IC705 78L005AP, Q701 ?, Q702 ?, Q705 ?

Commit message: prices and vaules. kicad wheres the 1P4S
Parts:
- added C725, C726: 10uF, symbol Device:C_Polarized
- added C727: 10nF, symbol Device:C
- added P1: Conn_WallPlug, symbol Connector:Conn_WallPlug
- C701: value 28 140K -> 100nF
- C705, C706, C707, C728: value ? -> 10nF
- C708: value ? -> 3,3mF; symbol Device:C -> Device:C_Polarized
- C709, C714: value ? -> 470uF; symbol Device:C -> Device:C_Polarized
- C711, C713: value ? -> 1mF; symbol Device:C -> Device:C_Polarized
- C712, C715, C717: value ? -> 220uF; symbol Device:C -> Device:C_Polarized
- C716, C724: value ? -> 330uF; symbol Device:C -> Device:C_Polarized
- C722: value ? -> 3,9nF
- C723: value ? -> 47uF; symbol Device:C -> Device:C_Polarized
- D701, D702, D703, D704: value ? -> 508
- D706: value ? -> 532
- D707: value ? -> 565
- D710: value ? -> 550
- IC705: value 78L005AP -> TA78L005AP
- Q701: value ? -> A935 QW; symbol Device:Q_NPN_CBE -> Device:Q_PNP_CBE
- Q702: value ? -> A957 98; symbol Device:Q_NPN_CBE -> Device:Q_PNP_CBE
- Q705: value ? -> D1812 QY
- R702, R703: value ? -> 1
- R704, R705: value ? -> 10k
- R706: value ? -> 270
- R707: value ? -> 15
- R708: value ? -> 120
- R712: value ? -> 3,9k
- R713: value ? -> 100
Connections:
- net BK_1: now also C725.2, C726.2, C727.1
- net BK_2: now also C726.1
- net DC_7: now also C727.2
- net at IC703.1 (Pin_1), R708.1: now also C725.1
- net AC_1: no longer names the net of F701.1
- net AC_1: now also P1.1 (AC_P)
- net AC_2: no longer names the net of C701.2, FL701.3
- net AC_2: now also P1.2 (AC_N)
Other:
- note added: "0.8"
- note added: "2022-11-24"
- note added: "Author: svp CC0"
- note added: "PWBF5790CE (P5789CE)"
- note added: "SHARP RGB SYSTEM TUNER CZ-6TU - PSU BOARD"
- note added: "T701 KICAD WHERE IS THE 1P4S TRANSFORMER ZEBRA DBP-57-28A / 4 PO454CE 13QOZK"
- note removed: "T701 THIS PIECE OF #### PHYSICALLY BENDS THE BOARD ZEBRA DBP-57-28A / 4 PO454CE 13QOZK"
- moved on the sheet: IC703, Q705

Commit message: partial cleanup, hopefully fixed some symbols
Parts:
- removed IC701, IC702: 78012AP, symbol Connector_Generic:Conn_01x03
- removed IC703: 78005AP, symbol Connector_Generic:Conn_01x03
- removed IC704: 78009AP, symbol Connector_Generic:Conn_01x03
- removed IC705: TA78L005AP, symbol Connector_Generic:Conn_01x03
- added IC701, IC702: TA78012AP, symbol Regulator_Linear:L7812
- added IC703, IC705: TA78005AP, symbol Regulator_Linear:L7805
- added IC704: TA78009AP, symbol Regulator_Linear:L7809
Connections:
- net BK_1: now also IC701.2 (GND), IC702.2 (GND), IC703.2 (GND), IC704.2 (GND), IC705.2 (GND)
- net BK_3: now also IC705.3 (OUT)
- net BK_5: now also R713.1, IC701.3 (OUT); no longer R713.2
- net DC_4: now also IC704.3 (OUT)
- net DC_5: now also IC702.3 (OUT)
- net DC_6: now also IC703.3 (OUT)
- net DC_7: no longer C713.1, C727.2, R705.2, R707.1, R708.2
- net at C723.1: now also R713.2, IC705.1 (IN); no longer R713.1
- net at C725.1, R708.1: now also IC703.1 (IN)
- net at C711.1, D706.1 (K): now also IC701.1 (IN)
- new net: C713.1, C727.2, IC702.1 (IN), IC704.1 (IN), R705.2, R707.1, R708.2
- no-connect marks 0 -> 8
Other:
- note added: "0.81"
- note added: "T701 1P4S TRANSFORMER ZEBRA DBP-57-28A / 4 PO454CE 13QOZK"
- note removed: "0.8"
- note removed: "T701 KICAD WHERE IS THE 1P4S TRANSFORMER ZEBRA DBP-57-28A / 4 PO454CE 13QOZK"
- moved on the sheet: C712, C713, C714, C715, C717, C723, C727, Q702, Q705, R707, R708, R713
